Commit message: convert stl to obj

File: urdf/g1_description/g1_23dof.urdf (robot description, URDF)
Before this commit: robot g1_23dof, 33 links, 32 joints
Links:
- link head_link: geometry collision mesh filename=meshes/head_link.obj; visual mesh filename=meshes/head_link.obj
- link left_ankle_pitch_link: geometry collision mesh filename=meshes/left_ankle_pitch_link.obj; visual mesh filename=meshes/left_ankle_pitch_link.obj
- link left_ankle_roll_link: geometry collision sphere radius=0.005; collision sphere radius=0.005
- link left_elbow_link: geometry collision mesh filename=meshes/left_elbow_link.obj; visual mesh filename=meshes/left_elbow_link.obj
- link left_hip_pitch_link: geometry collision mesh filename=meshes/left_hip_pitch_link.obj; visual mesh filename=meshes/left_hip_pitch_link.obj
- link left_hip_roll_link: geometry collision mesh filename=meshes/left_hip_roll_link.obj; visual mesh filename=meshes/left_hip_roll_link.obj
- link left_hip_yaw_link: geometry collision mesh filename=meshes/left_hip_yaw_link.obj; visual mesh filename=meshes/left_hip_yaw_link.obj
- link left_knee_link: geometry collision mesh filename=meshes/left_knee_link.obj; visual mesh filename=meshes/left_knee_link.obj
- link left_shoulder_pitch_link: geometry collision cylinder length=0.05 radius=0.03; visual mesh filename=meshes/left_shoulder_pitch_link.obj
- link left_shoulder_roll_link: geometry collision cylinder length=0.03 radius=0.03; visual mesh filename=meshes/left_shoulder_roll_link.obj
- link left_shoulder_yaw_link: geometry collision mesh filename=meshes/left_shoulder_yaw_link.obj; visual mesh filename=meshes/left_shoulder_yaw_link.obj
- link left_wrist_roll_rubber_hand: geometry collision mesh filename=meshes/left_wrist_roll_rubber_hand.obj; visual mesh filename=meshes/left_wrist_roll_rubber_hand.obj
- link logo_link: geometry collision mesh filename=meshes/logo_link.obj; visual mesh filename=meshes/logo_link.obj
- link pelvis: geometry visual mesh filename=meshes/pelvis.obj
- link pelvis_contour_link: geometry collision mesh filename=meshes/pelvis_contour_link.obj; visual mesh filename=meshes/pelvis_contour_link.obj
- link right_ankle_pitch_link: geometry collision mesh filename=meshes/right_ankle_pitch_link.obj; visual mesh filename=meshes/right_ankle_pitch_link.obj
- link right_ankle_roll_link: geometry collision sphere radius=0.005; collision sphere radius=0.005
- link right_elbow_link: geometry collision mesh filename=meshes/right_elbow_link.obj; visual mesh filename=meshes/right_elbow_link.obj
- link right_hip_pitch_link: geometry collision mesh filename=meshes/right_hip_pitch_link.obj; visual mesh filename=meshes/right_hip_pitch_link.obj
- link right_hip_roll_link: geometry collision mesh filename=meshes/right_hip_roll_link.obj; visual mesh filename=meshes/right_hip_roll_link.obj
- link right_hip_yaw_link: geometry collision mesh filename=meshes/right_hip_yaw_link.obj; visual mesh filename=meshes/right_hip_yaw_link.obj
- link right_knee_link: geometry collision mesh filename=meshes/right_knee_link.obj; visual mesh filename=meshes/right_knee_link.obj
- link right_shoulder_pitch_link: geometry collision cylinder length=0.05 radius=0.03; visual mesh filename=meshes/right_shoulder_pitch_link.obj
- link right_shoulder_roll_link: geometry collision cylinder length=0.03 radius=0.03; visual mesh filename=meshes/right_shoulder_roll_link.obj
- link right_shoulder_yaw_link: geometry collision mesh filename=meshes/right_shoulder_yaw_link.obj; visual mesh filename=meshes/right_shoulder_yaw_link.obj
- link right_wrist_roll_rubber_hand: geometry collision mesh filename=meshes/right_wrist_roll_rubber_hand.obj; visual mesh filename=meshes/right_wrist_roll_rubber_hand.obj
- link torso_link: geometry collision mesh filename=meshes/torso_link.obj; visual mesh filename=meshes/torso_link.obj
- link waist_support_link: geometry collision mesh filename=meshes/waist_support_link.obj; visual mesh filename=meshes/waist_support_link.obj
- link waist_yaw_fixed_link: geometry visual mesh filename=meshes/waist_yaw_link.obj
